File: hardware/HumidityLoggerBreakout/_autosave-HumidityLoggerBreakout.kicad_pcb (KiCad board)
At the start: 2 copper layers, 98 x 74 mm, 45 parts, among them J1 PWR_IN, J2 BME280, J3 +5V_OUT, J4 IO, J6 Conn_01x11, J7 Conn_01x11, J8 I2C_MCU, U1 LM317_TO-252

Commit message: WIP of the new version.
Parts:
- J6, J7: footprint Connector_PinHeader_2.54mm:PinHeader_1x11_P2.54mm_Vertical -> Connector_PinSocket_2.54mm:PinSocket_1x11_P2.54mm_Vertical
- J8: footprint Connector_PinHeader_2.54mm:PinHeader_1x04_P2.54mm_Vertical -> Connector_PinSocket_2.54mm:PinSocket_1x04_P2.54mm_Vertical
