File: hardware/HumidityLoggerBreakout/HumidityLoggerBreakout.kicad_sch (KiCad schematic)
At the start: 43 parts, among them J1 Barrel_Jack_Switch, J10 RELAY_PWR, J2 POWER_IN, J3 LEVEL, J4 RELAY, J5 MCU_PWR, J6 Conn_01x11, J7 Conn_01x11, J8 I2C, J9 I2C_OUT, U1 LM317_TO-252

Commit message: First prototype production files.
Parts:
- C1, C10, C11, C2: LCSC (none) -> C45783
- C12, C3, C4, C6, C7, C8, C9: LCSC (none) -> C28233
- C5: LCSC (none) -> C16133
- D1, D3, D4: LCSC (none) -> C2297
- D2: LCSC (none) -> C2296
- D5: LCSC (none) -> C84256
- J1, J10, J2, J3, J4, J5, J6, J7, J8, J9: LCSC (none) -> -
- R1, R2, R3, R4: LCSC (none) -> C17604
- R10, R12, R13, R14, R15, R5, R6, R7, R8, R9: LCSC (none) -> C17513
- R11: LCSC (none) -> C17630
- U1: LCSC (none) -> C75510
Changed lines of the file:
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@@
+      (effects (font (size 1.27 1.27)) hide)
+    )
+    (property "LCSC" "C28233" (id 4) (at 148.59 83.82 0)
       (effects (font (size 1.27 1.27)) hide)
     )
@@
     )
     (property "Datasheet" "~" (id 3) (at 162.56 83.82 0)
+      (effects (font (size 1.27 1.27)) hide)
+    )
+    (property "LCSC" "C28233" (id 4) (at 162.56 83.82 0)
       (effects (font (size 1.27 1.27)) hide)
     )
@@
       (effects (font (size 1.27 1.27)) hide)
     )
+    (property "LCSC" "C45783" (id 4) (at 77.47 109.22 0)
+      (effects (font (size 1.27 1.27)) hide)
+    )
     (pin "1")
     (pin "2")
@@
     )
     (property "Datasheet" "~" (id 3) (at 188.595 83.82 0)
+      (effects (font (size 1.27 1.27)) hide)
+    )
+    (property "LCSC" "C28233" (id 4) (at 188.595 83.82 0)
       (effects (font (size 1.27 1.27)) hide)
     )
@@
       (effects (font (size 1.27 1.27)) hide)
     )
+    (property "LCSC" "C28233" (id 4) (at 116.84 109.22 0)
+      (effects (font (size 1.27 1.27)) hide)
+    )
     (pin "1")
     (pin "2")
@@
     )
     (property "Datasheet" "~" (id 3) (at 146.05 158.75 0)
+      (effects (font (size 1.27 1.27)) hide)
+    )
+    (property "LCSC" "-" (id 4) (at 146.05 158.75 0)
       (effects (font (size 1.27 1.27)) hide)
     )
@@
       (effects (font (size 1.27 1.27)) hide)
     )
+    (property "LCSC" "C84256" (id 4) (at 200.025 57.15 0)
+      (effects (font (size 1.27 1.27)) hide)
+    )
     (pin "1")
     (pin "2")
@@
       (effects (font (size 1.27 1.27)) hide)
     )
+    (property "LCSC" "-" (id 4) (at 242.57 87.63 0)
+      (effects (font (size 1.27 1.27)) hide)
+    )
     (pin "1")
     (pin "2")
@@
       (effects (font (size 1.27 1.27)) hide)
     )
+    (property "LCSC" "C17513" (id 4) (at 105.41 58.42 0)
+      (effects (font (size 1.27 1.27)) hide)
+    )
     (pin "1")
     (pin "2")
@@
     )
     (property "Datasheet" "~" (id 3) (at 137.16 123.19 0)
+      (effects (font (size 1.27 1.27)) hide)
+    )
+    (property "LCSC" "C2297" (id 4) (at 137.16 123.19 0)
       (effects (font (size 1.27 1.27)) hide)
     )
@@
       (effects (font (size 1.27 1.27)) hide)
     )
+    (property "LCSC" "C17513" (id 4) (at 67.31 146.05 0)
+      (effects (font (size 1.27 1.27)) hide)
+    )
     (pin "1")
     (pin "2")
@@
       (effects (font (size 1.27 1.27)) hide)
     )
+    (property "LCSC" "C17513" (id 4) (at 67.31 138.43 0)
+      (effects (font (size 1.27 1.27)) hide)
+    )
     (pin "1")
     (pin "2")
@@
     )
     (property "Datasheet" "~" (id 3) (at 184.785 122.555 0)
+      (effects (font (size 1.27 1.27)) hide)
+    )
+    (property "LCSC" "C17513" (id 4) (at 184.785 122.555 0)
       (effects (font (size 1.27 1.27)) hide)
     )
@@
       (effects (font (size 1.27 1.27)) hide)
     )
+    (property "LCSC" "-" (id 4) (at 36.83 77.47 0)
+      (effects (font (size 1.27 1.27)) hide)
+    )
     (pin "1")
     (pin "2")
@@
     )
     (property "Datasheet" "~" (id 3) (at 200.025 67.31 0)
+      (effects (font (size 1.27 1.27)) hide)
+    )
+    (property "LCSC" "C17513" (id 4) (at 200.025 67.31 0)
       (effects (font (size 1.27 1.27)) hide)
     )
@@
       (effects (font (size 1.27 1.27)) hide)
     )
+    (property "LCSC" "C17513" (id 4) (at 67.31 154.305 0)
+      (effects (font (size 1.27 1.27)) hide)
+    )
     (pin "1")
     (pin "2")
@@
     )
     (property "Datasheet" "~" (id 3) (at 38.1 107.95 0)
+      (effects (font (size 1.27 1.27)) hide)
+    )
+    (property "LCSC" "-" (id 4) (at 38.1 107.95 0)
       (effects (font (size 1.27 1.27)) hide)
     )
@@
       (effects (font (size 1.27 1.27)) hide)
     )
+    (property "LCSC" "C75510" (id 4) (at 101.6 92.075 0)
+      (effects (font (size 1.27 1.27)) hide)
+    )
     (pin "1")
     (pin "2")
@@
     )
     (property "Datasheet" "~" (id 3) (at 128.27 109.22 0)
+      (effects (font (size 1.27 1.27)) hide)
+    )
+    (property "LCSC" "C16133" (id 4) (at 128.27 109.22 0)
       (effects (font (size 1.27 1.27)) hide)
     )
@@
       (effects (font (size 1.27 1.27)) hide)
     )
+    (property "LCSC" "C17513" (id 4) (at 101.6 107.315 0)
+      (effects (font (size 1.27 1.27)) hide)
+    )
     (pin "1")
     (pin "2")
@@
     )
     (property "Datasheet" "~" (id 3) (at 242.57 118.11 0)
+      (effects (font (size 1.27 1.27)) hide)
+    )
+    (property "LCSC" "-" (id 4) (at 242.57 118.11 0)
       (effects (font (size 1.27 1.27)) hide)
     )
@@
       (effects (font (size 1.27 1.27)) hide)
     )
+    (property "LCSC" "-" (id 4) (at 163.83 113.03 0)
+      (effects (font (size 1.27 1.27)) hide)
+    )
     (pin "1")
     (pin "2")
@@
     )
     (property "Datasheet" "~" (id 3) (at 96.52 160.02 0)
+      (effects (font (size 1.27 1.27)) hide)
+    )
+    (property "LCSC" "-" (id 4) (at 96.52 160.02 0)
       (effects (font (size 1.27 1.27)) hide)
     )
@@
       (effects (font (size 1.27 1.27)) hide)
     )
+    (property "LCSC" "C17513" (id 4) (at 67.31 130.81 0)
+      (effects (font (size 1.27 1.27)) hide)
+    )
     (pin "1")
     (pin "2")
@@
     )
     (property "Datasheet" "~" (id 3) (at 87.63 109.22 0)
+      (effects (font (size 1.27 1.27)) hide)
+    )
+    (property "LCSC" "C28233" (id 4) (at 87.63 109.22 0)
       (effects (font (size 1.27 1.27)) hide)
     )
@@
       (effects (font (size 1.27 1.27)) hide)
     )
+    (property "LCSC" "C17630" (id 4) (at 110.49 102.87 0)
+      (effects (font (size 1.27 1.27)) hide)
+    )
     (pin "1")
     (pin "2")
@@
       (effects (font (size 1.27 1.27)) hide)
     )
+    (property "LCSC" "C17604" (id 4) (at 39.37 169.545 0)
+      (effects (font (size 1.27 1.27)) hide)
+    )
     (pin "1")
     (pin "2")
@@
       (effects (font (size 1.27 1.27)) hide)
     )
+    (property "LCSC" "C28233" (id 4) (at 233.68 146.685 0)
+      (effects (font (size 1.27 1.27)) hide)
+    )
     (pin "1")
     (pin "2")
@@
     )
     (property "Datasheet" "~" (id 3) (at 118.745 58.42 0)
+      (effects (font (size 1.27 1.27)) hide)
+    )
+    (property "LCSC" "C17513" (id 4) (at 118.745 58.42 0)
       (effects (font (size 1.27 1.27)) hide)
     )
@@
       (effects (font (size 1.27 1.27)) hide)
     )
+    (property "LCSC" "C2297" (id 4) (at 184.785 133.985 0)
+      (effects (font (size 1.27 1.27)) hide)
+    )
     (pin "1")
     (pin "2")
@@
       (effects (font (size 1.27 1.27)) hide)
     )
+    (property "LCSC" "C17513" (id 4) (at 137.16 111.76 0)
+      (effects (font (size 1.27 1.27)) hide)
+    )
     (pin "1")
     (pin "2")
@@
     )
     (property "Datasheet" "~" (id 3) (at 105.41 48.26 0)
+      (effects (font (size 1.27 1.27)) hide)
+    )
+    (property "LCSC" "C2297" (id 4) (at 105.41 48.26 0)
       (effects (font (size 1.27 1.27)) hide)
     )
@@
       (effects (font (size 1.27 1.27)) hide)
     )
+    (property "LCSC" "C45783" (id 4) (at 66.04 108.585 0)
+      (effects (font (size 1.27 1.27)) hide)
+    )
     (pin "1")
     (pin "2")
@@
       (effects (font (size 1.27 1.27)) hide)
     )
+    (property "LCSC" "C17604" (id 4) (at 46.355 169.545 0)
+      (effects (font (size 1.27 1.27)) hide)
+    )
     (pin "1")
     (pin "2")
@@
     )
     (property "Datasheet" "~" (id 3) (at 176.53 49.53 0)
+      (effects (font (size 1.27 1.27)) hide)
+    )
+    (property "LCSC" "-" (id 4) (at 176.53 49.53 0)
       (effects (font (size 1.27 1.27)) hide)
     )
@@
       (effects (font (size 1.27 1.27)) hide)
     )
+    (property "LCSC" "C17604" (id 4) (at 60.325 169.545 0)
+      (effects (font (size 1.27 1.27)) hide)
+    )
     (pin "1")
     (pin "2")
@@
       (effects (font (size 1.27 1.27)) hide)
     )
+    (property "LCSC" "C2296" (id 4) (at 118.745 48.26 0)
+      (effects (font (size 1.27 1.27)) hide)
+    )
     (pin "1")
     (pin "2")
@@
       (effects (font (size 1.27 1.27)) hide)
     )
+    (property "LCSC" "C17604" (id 4) (at 53.34 169.545 0)
+      (effects (font (size 1.27 1.27)) hide)
+    )
     (pin "1")
     (pin "2")
@@
       (effects (font (size 1.27 1.27)) hide)
     )
+    (property "LCSC" "C28233" (id 4) (at 175.26 83.82 0)
+      (effects (font (size 1.27 1.27)) hide)
+    )
     (pin "1")
     (pin "2")
@@
     )
     (property "Datasheet" "~" (id 3) (at 207.645 146.05 0)
+      (effects (font (size 1.27 1.27)) hide)
+    )
+    (property "LCSC" "C45783" (id 4) (at 207.645 146.05 0)
       (effects (font (size 1.27 1.27)) hide)
     )
@@
       (effects (font (size 1.27 1.27)) hide)
     )
+    (property "LCSC" "C45783" (id 4) (at 220.345 146.685 0)
+      (effects (font (size 1.27 1.27)) hide)
+    )
     (pin "1")
     (pin "2")
@@
       (effects (font (size 1.27 1.27)) hide)
     )
+    (property "LCSC" "-" (id 4) (at 251.46 146.685 0)
+      (effects (font (size 1.27 1.27)) hide)
+    )
     (pin "1")
     (pin "2")
@@
       (effects (font (size 1.27 1.27)) hide)
     )
+    (property "LCSC" "-" (id 4) (at 241.3 49.53 0)
+      (effects (font (size 1.27 1.27)) hide)
+    )

Commit message: Modified the schematic to drop unnecessary features.
Parts:
- removed J3: LEVEL, Connector_PinHeader_2.54mm:PinHeader_1x06_P2.54mm_Vertical, symbol Connector_Generic:Conn_01x06
- removed J5: MCU_PWR, Connector_PinHeader_2.54mm:PinHeader_1x02_P2.54mm_Vertical, symbol Connector_Generic:Conn_01x02
- added D6: LOW, LED_SMD:LED_0805_2012Metric_Pad1.15x1.40mm_HandSolder, symbol Device:D_Filled
- added D7: OK, LED_SMD:LED_0805_2012Metric_Pad1.15x1.40mm_HandSolder, symbol Device:D_Filled
- added D8: HIGH, LED_SMD:LED_0805_2012Metric_Pad1.15x1.40mm_HandSolder, symbol Device:D_Filled
- added D9: VHIGH, LED_SMD:LED_0805_2012Metric_Pad1.15x1.40mm_HandSolder, symbol Device:D_Filled
- added J3: MCU_PWR, TerminalBlock_Phoenix:TerminalBlock_Phoenix_PT-1,5-2-3.5-H_1x02_P3.50mm_Horizontal, symbol Connector:Screw_Terminal_01x02
- J10: value RELAY_PWR -> PWR_OUT
- J2: value POWER_IN -> PWR_IN
- J4: value RELAY -> IO
- J8: value I2C -> I2C_MCU
- R1, R2, R3, R4: value 2k -> 1k; LCSC C17604 -> C17513
Connections:
- net +5V: now also J3.2 (Pin_2)
- net D10: no longer R1.2
- net D11: no longer R2.2
- net D12: no longer R3.2
- net D13: no longer R4.2
- net GND: now also R1.2, R2.2, R3.2, R4.2, J3.1 (Pin_1); no longer R1.1, R2.1, R3.1, R4.1
- net at R7.2: now also D7.2 (A)
- net at R6.2: now also D8.2 (A)
- net at R8.2: now also D6.2 (A)
- net at R5.2: now also D9.2 (A)
- new net: D6.1 (K), R1.1
- new net: D8.1 (K), R3.1
- new net: D9.1 (K), R4.1
- new net: D7.1 (K), R2.1
Other:
- moved on the sheet: J4

Commit message: WIP of the new version.
Parts:
- removed C10, C11: 22u, Capacitor_SMD:C_0805_2012Metric_Pad1.18x1.45mm_HandSolder, symbol Device:C
- removed C12: 100n, Capacitor_SMD:C_0805_2012Metric_Pad1.18x1.45mm_HandSolder, symbol Device:C
- removed D4: 3V3, LED_SMD:LED_0805_2012Metric_Pad1.15x1.40mm_HandSolder, symbol Device:D_Filled
- removed J10: PWR_OUT, TerminalBlock_Phoenix:TerminalBlock_Phoenix_PT-1,5-2-3.5-H_1x02_P3.50mm_Horizontal, symbol Connector:Screw_Terminal_01x02
- removed J2: PWR_IN, TerminalBlock_Phoenix:TerminalBlock_Phoenix_PT-1,5-2-3.5-H_1x02_P3.50mm_Horizontal, symbol Connector:Screw_Terminal_01x02
- removed J9: I2C_OUT, Connector_PinHeader_2.54mm:PinHeader_1x04_P2.54mm_Vertical, symbol Connector_Generic:Conn_01x04
- removed R1, R14, R2, R3, R4: 1k, Resistor_SMD:R_0805_2012Metric_Pad1.20x1.40mm_HandSolder, symbol Device:R
- added H1, H2, H3, H4: MountingHole_Pad, MountingHole:MountingHole_2.7mm_M2.5_Pad_TopBottom, symbol Mechanical:MountingHole_Pad
- added J2: BME280, Connector_PinHeader_2.54mm:PinHeader_1x06_P2.54mm_Vertical, symbol Connector_Generic:Conn_01x06
- D1: value LED1 -> MCU
- D2: value LED2 -> ACT
- D5: value LED3 -> ERR
- J1: value Barrel_Jack_Switch -> PWR_IN
- J3: value MCU_PWR -> +5V_OUT
- J6, J7: footprint Connector_PinHeader_2.54mm:PinHeader_1x11_P2.54mm_Vertical -> Connector_PinSocket_2.54mm:PinSocket_1x11_P2.54mm_Vertical
- J8: footprint Connector_PinHeader_2.54mm:PinHeader_1x04_P2.54mm_Vertical -> Connector_PinSocket_2.54mm:PinSocket_1x04_P2.54mm_Vertical
Connections:
- net +3.3V: now also J2.1 (Pin_1)
- net GND: now also D6.1 (K), D7.1 (K), D8.1 (K), D9.1 (K), H1.1, H2.1, H3.1, H4.1, J2.2 (Pin_2)
- net SCL: now also J2.3 (Pin_3)
- net SDA: now also J2.4 (Pin_4)
- no-connect marks 11 -> 13

Commit message: WIP on the board.
Parts:
- removed C2: 22u, Capacitor_SMD:C_0805_2012Metric_Pad1.18x1.45mm_HandSolder, symbol Device:C
- removed C3, C4, C6, C7, C8: 100n, Capacitor_SMD:C_0805_2012Metric_Pad1.18x1.45mm_HandSolder, symbol Device:C
- removed C5: 100u, Capacitor_Tantalum_SMD:CP_EIA-3528-12_Kemet-T_Pad1.50x2.35mm_HandSolder, symbol Device:C_Polarized
- removed D3: 5V, LED_SMD:LED_0805_2012Metric_Pad1.15x1.40mm_HandSolder, symbol Device:D_Filled
- removed J1: PWR_IN, Connector_BarrelJack:BarrelJack_Horizontal, symbol Connector:Barrel_Jack_Switch
- removed J3: +5V_OUT, TerminalBlock_Phoenix:TerminalBlock_Phoenix_PT-1,5-2-3.5-H_1x02_P3.50mm_Horizontal, symbol Connector:Screw_Terminal_01x02
- removed R11: 330, Resistor_SMD:R_0805_2012Metric_Pad1.20x1.40mm_HandSolder, symbol Device:R
- removed R13, R9: 1k, Resistor_SMD:R_0805_2012Metric_Pad1.20x1.40mm_HandSolder, symbol Device:R
- removed U1: LM317_TO-252, Package_TO_SOT_SMD:TO-252-2, symbol Regulator_Linear:LM317_TO-252
- renumbered C9 to C2, D6 to D1, D7 to D2, D8 to D3, D9 to D4, D1 to D5, D2 to D6, D5 to D7, J4 to J1, J6 to J2, J8 to J3, J2 to J4, J7 to J5, R5 to R1, R6 to R2, R7 to R3, R8 to R4, R10 to R5, R12 to R6, R15 to R7
Connections:
- net +12V is gone; now on net +3.3V: C1.1
- net +3.3V: now also J1.1 (Pin_1)
- net +5V: no longer J1.1 (Pin_1)
- no-connect marks 13 -> 12
Other:
- moved on the sheet: D5, D6, D7, J2, J5, R5, R6, R7
